Commit message: added ex01

File: ex01/gazebo_robot/robot.gazebo.xacro (robot description, xacro)
@@ -2,5 +2,4 @@
 <robot xmlns:xacro="http://www.ros.org/wiki/xacro">
     <gazebo>
-        <!-- Плагин для состояния суставов -->
         <plugin
             filename="libgz-sim-joint-state-publisher-system.so"
@@ -12,9 +11,7 @@
             <update_rate>50</update_rate>
         </plugin>
-        <!-- Плагин для дифференциального привода -->
         <plugin
             filename="libgz-sim-diff-drive-system.so"
             name="gz::sim::systems::DiffDrive">
-            <!-- Укажите ВСЕ колесные суставы -->
             <left_joint>left_front_wheel_joint</left_joint>
             <left_joint>left_back_wheel_joint</left_joint>
@@ -24,5 +21,5 @@
             <wheel_radius>0.035</wheel_radius>
             <odom_publish_frequency>30</odom_publish_frequency>
-            <topic>/model/robot/cmd_vel</topic>
+            <topic>/cmd_vel</topic>
         </plugin>
     </gazebo>

File: ex01/gazebo_robot/robot.urdf.xacro (robot description, xacro)
@@ -1,4 +1,5 @@
 <?xml version="1.0"?>
 <robot name="visual_robot" xmlns:xacro="http://www.ros.org/wiki/xacro">
+  <xacro:include filename="$(find gazebo_robot)/robot.gazebo.xacro" />
   <!-- Константы -->
   <xacro:property name="M_PI" value="3.1415926535897931" />
@@ -179,5 +180,27 @@
     <origin xyz="0.1814 0 0.1414"/>
   </joint>
-  <!-- Gazebo plugins -->
+  <joint name="lidar_joint" type="fixed">
+    <parent link="base_link"/>
+    <child link="lidar_link"/>
+    <origin xyz="0.2 0 0.22" rpy="0 0 0"/>
+  </joint>
+  <link name="lidar_link">
+    <visual>
+      <geometry>
+        <cylinder radius="0.05" length="0.04"/>
+      </geometry>
+      <material name="black"/>
+    </visual>
+    <collision>
+      <geometry>
+        <cylinder radius="0.05" length="0.04"/>
+      </geometry>
+    </collision>
+    <inertial>
+      <mass value="0.1"/>
+      <inertia ixx="0.0001" ixy="0" ixz="0" iyy="0.0001" iyz="0" izz="0.0001"/>
+    </inertial>
+  </link>
+  <!-- Gazebo plugins
   <gazebo>
     <plugin filename="libgz-sim-diff-drive-system.so" name="gz::sim::systems::DiffDrive">
@@ -191,4 +214,28 @@
       <topic>/model/robot/cmd_vel</topic>
     </plugin>
+  </gazebo> -->
+  <gazebo reference="lidar_link">
+    <sensor name="lidar" type="gpu_lidar">
+      <pose>0 0 0 0 0 0</pose>
+      <topic>scan</topic>
+      <update_rate>10</update_rate>
+      <gz_frame_id>lidar_link</gz_frame_id>
+      <visualize>false</visualize>
+      <ray>
+        <scan>
+          <horizontal>
+            <samples>180</samples>
+            <resolution>1</resolution>
+            <min_angle>-3.14159</min_angle>
+            <max_angle>3.14159</max_angle>
+          </horizontal>
+        </scan>
+        <range>
+          <min>0.15</min>
+          <max>10.0</max>
+        </range>
+      </ray>
+      <always_on>1</always_on>
+    </sensor>
   </gazebo>
   <!-- Gazebo materials (для симуляции) -->
